File: hw/main.sch (EAGLE design)
At the start: 22 parts, among them T1 PMBT4401,215, T2 PMBT4401,215, U1 MCP1703T-3002E/CB, U2 MSP430G2452IPW14R, U3 TCS3414CS, X1 DF13-4P-1.25V(50), X2 DF13-4P-1.25V(50)

Commit message: Fix errors in PCB found after initial testing.
 - Swapped pullup/down on RST/TEST lines (they were backward).
 - Added 4.7k pullups to i2c lines (maybe don't need but the signal is a little ugly without them)
 - Removed silkscreen of part numbers since they're not very readable anyway
Parts:
- added R10, R9: RK73H1JTTD4701F, rcl:R-US_R0603
Connections:
- net +3V3: now also R10.2, R9.2
- net CLK: now also R10.1
- net DAT: now also R9.1
- net RST: now also R1.1; no longer R2.2
- net TEST: now also R2.2; no longer R1.1
Other:
- note removed: "Programming Connector"
- moved on the sheet: R1, R2
Changed lines of the file:
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@@
 <setting verticaltext="up"/>
 </settings>
-<grid distance="0.1" unitdist="inch" unit="inch" style="lines" multiple="1" display="no" altdistance="0.01" altunitdist="inch" altunit="inch"/>
+<grid distance="0.1" unitdist="inch" unit="inch" style="lines" multiple="1" display="yes" altdistance="0.01" altunitdist="inch" altunit="inch"/>
 <layers>
 <layer number="1" name="Top" color="4" fill="1" visible="no" active="no"/>
@@
 <part name="X2" library="con-molex" deviceset="53?-04" device="398" value="DF13-4P-1.25V(50)"/>
 <part name="X1" library="con-molex" deviceset="53?-04" device="398" value="DF13-4P-1.25V(50)"/>
+<part name="R9" library="rcl" deviceset="R-US_" device="R0603" value="RK73H1JTTD4701F"/>
+<part name="R10" library="rcl" deviceset="R-US_" device="R0603" value="RK73H1JTTD4701F"/>
+<part name="+3V2" library="supply1" deviceset="+3V3" device=""/>
+<part name="+3V8" library="supply1" deviceset="+3V3" device=""/>
 </parts>
 <sheets>
 <sheet>
 <plain>
-<text x="2.54" y="50.8" size="2.54" layer="97">Programming Connector</text>
 <wire x1="0" y1="0" x2="53.34" y2="0" width="0.1524" layer="97" style="longdash"/>
 <wire x1="53.34" y1="0" x2="149.86" y2="0" width="0.1524" layer="97" style="longdash"/>
@@
 <attribute name="VALUE" x="165.1" y="101.6" size="2.54" layer="96"/>
 </instance>
-<instance part="R1" gate="G$1" x="12.7" y="35.56" smashed="yes" rot="R90">
-<attribute name="NAME" x="7.62" y="35.56" size="2.54" layer="95"/>
-</instance>
-<instance part="R2" gate="G$1" x="12.7" y="22.86" smashed="yes" rot="R90">
-<attribute name="NAME" x="7.62" y="22.86" size="2.54" layer="95"/>
-</instance>
-<instance part="GND8" gate="1" x="12.7" y="12.7" smashed="yes">
-<attribute name="VALUE" x="10.16" y="10.16" size="2.54" layer="96"/>
-</instance>
-<instance part="+3V7" gate="G$1" x="12.7" y="45.72" smashed="yes">
-<attribute name="VALUE" x="10.16" y="45.72" size="2.54" layer="96"/>
+<instance part="R1" gate="G$1" x="25.4" y="38.1" smashed="yes" rot="R90">
+<attribute name="NAME" x="20.32" y="38.1" size="2.54" layer="95"/>
+</instance>
+<instance part="R2" gate="G$1" x="17.78" y="22.86" smashed="yes" rot="R90">
+<attribute name="NAME" x="12.7" y="22.86" size="2.54" layer="95"/>
+</instance>
+<instance part="GND8" gate="1" x="17.78" y="12.7" smashed="yes">
+<attribute name="VALUE" x="15.24" y="10.16" size="2.54" layer="96"/>
+</instance>
+<instance part="+3V7" gate="G$1" x="25.4" y="45.72" smashed="yes">
+<attribute name="VALUE" x="22.86" y="45.72" size="2.54" layer="96"/>
 </instance>
 <instance part="U3" gate="G$1" x="195.58" y="22.86" smashed="yes">
@@
 </instance>
 <instance part="T2" gate="G$1" x="187.96" y="71.12" smashed="yes">
-<attribute name="NAME" x="193.04" y="76.2" size="2.54" layer="95"/>
+<attribute name="NAME" x="193.04" y="71.12" size="2.54" layer="95"/>
 </instance>
 <instance part="R8" gate="G$1" x="180.34" y="71.12" smashed="yes" rot="R180">
@@
 <instance part="X1" gate="-4" x="236.22" y="66.04" smashed="yes" rot="MR0">
 <attribute name="NAME" x="233.68" y="65.278" size="2.54" layer="95" rot="MR0"/>
+</instance>
+<instance part="R9" gate="G$1" x="175.26" y="40.64" smashed="yes" rot="R90">
+<attribute name="NAME" x="170.18" y="40.64" size="2.54" layer="95"/>
+</instance>
+<instance part="R10" gate="G$1" x="165.1" y="40.64" smashed="yes" rot="R90">
+<attribute name="NAME" x="160.02" y="40.64" size="2.54" layer="95"/>
+</instance>
+<instance part="+3V2" gate="G$1" x="175.26" y="48.26" smashed="yes">
+<attribute name="VALUE" x="172.72" y="48.26" size="2.54" layer="96"/>
+</instance>
+<instance part="+3V8" gate="G$1" x="165.1" y="48.26" smashed="yes">
+<attribute name="VALUE" x="162.56" y="48.26" size="2.54" layer="96"/>
 </instance>
 </instances>
@@
 <pinref part="R2" gate="G$1" pin="1"/>
 <pinref part="GND8" gate="1" pin="GND"/>
-<wire x1="12.7" y1="17.78" x2="12.7" y2="15.24" width="0.1524" layer="91"/>
+<wire x1="17.78" y1="17.78" x2="17.78" y2="15.24" width="0.1524" layer="91"/>
 </segment>
 <segment>
@@
 <pinref part="R1" gate="G$1" pin="2"/>
 <pinref part="+3V7" gate="G$1" pin="+3V3"/>
-<wire x1="12.7" y1="40.64" x2="12.7" y2="43.18" width="0.1524" layer="91"/>
 </segment>
 <segment>
@@
 <pinref part="U2" gate="G$1" pin="1"/>
 <wire x1="76.2" y1="35.56" x2="78.74" y2="35.56" width="0.1524" layer="91"/>
+</segment>
+<segment>
+<pinref part="R9" gate="G$1" pin="2"/>
+<pinref part="+3V2" gate="G$1" pin="+3V3"/>
+</segment>
+<segment>
+<pinref part="R10" gate="G$1" pin="2"/>
+<pinref part="+3V8" gate="G$1" pin="+3V3"/>
 </segment>
 </net>
@@
 <segment>
 <pinref part="U3" gate="G$1" pin="SDA"/>
-<wire x1="177.8" y1="27.94" x2="160.02" y2="27.94" width="0.1524" layer="91"/>
+<wire x1="177.8" y1="27.94" x2="175.26" y2="27.94" width="0.1524" layer="91"/>
 <label x="160.02" y="27.94" size="2.54" layer="95"/>
+<pinref part="R9" gate="G$1" pin="1"/>
+<wire x1="175.26" y1="27.94" x2="160.02" y2="27.94" width="0.1524" layer="91"/>
+<wire x1="175.26" y1="35.56" x2="175.26" y2="27.94" width="0.1524" layer="91"/>
+<junction x="175.26" y="27.94"/>
 </segment>
 <segment>
@@
 <segment>
 <pinref part="U3" gate="G$1" pin="SCL"/>
-<wire x1="177.8" y1="30.48" x2="160.02" y2="30.48" width="0.1524" layer="91"/>
+<wire x1="177.8" y1="30.48" x2="165.1" y2="30.48" width="0.1524" layer="91"/>
 <label x="160.02" y="30.48" size="2.54" layer="95"/>
+<pinref part="R10" gate="G$1" pin="1"/>
+<wire x1="165.1" y1="30.48" x2="160.02" y2="30.48" width="0.1524" layer="91"/>
+<wire x1="165.1" y1="35.56" x2="165.1" y2="30.48" width="0.1524" layer="91"/>
+<junction x="165.1" y="30.48"/>
 </segment>
 <segment>
@@
 </segment>
 <segment>
-<wire x1="30.48" y1="30.48" x2="12.7" y2="30.48" width="0.1524" layer="91"/>
-<label x="17.78" y="30.48" size="2.54" layer="95"/>
-<pinref part="R1" gate="G$1" pin="1"/>
 <pinref part="JP1" gate="G$1" pin="1"/>
+<pinref part="R2" gate="G$1" pin="2"/>
+<wire x1="30.48" y1="30.48" x2="17.78" y2="30.48" width="0.1524" layer="91"/>
+<wire x1="17.78" y1="30.48" x2="17.78" y2="27.94" width="0.1524" layer="91"/>
+<label x="17.78" y="30.48" size="1.778" layer="95"/>
 </segment>
 </net>
@@
 </segment>
 <segment>
-<wire x1="30.48" y1="27.94" x2="12.7" y2="27.94" width="0.1524" layer="91"/>
-<label x="17.78" y="27.94" size="2.54" layer="95"/>
-<pinref part="R2" gate="G$1" pin="2"/>
+<pinref part="R1" gate="G$1" pin="1"/>
+<wire x1="25.4" y1="33.02" x2="25.4" y2="27.94" width="0.1524" layer="91"/>
 <pinref part="JP1" gate="G$1" pin="2"/>
-</segment>
-</net>
+<wire x1="25.4" y1="27.94" x2="30.48" y2="27.94" width="0.1524" layer="91"/>
+<label x="25.4" y="27.94" size="1.778" layer="95"/>
+</segment>
+</net>
